File: hardware/micro_sheet.sch (KiCad schematic (older format))
At the start: 9 parts, among them IC1 ATTINY2313A-S, P5 CONN_3X2, SW1 SW_PUSH, X1 20MHz

Commit message: Added schematic for external temp sensor board. Updated netlists.
Connections:
- wire segments 53 -> 47
Changed lines of the file:
@@
-EESchema Schematic File Version 2  date Tue 18 Dec 2012 11:55:45 PM EST
+EESchema Schematic File Version 2  date Wed 19 Dec 2012 12:08:27 AM EST
 LIBS:power
 LIBS:device
@@
 $EndDescr
 $Comp
-L GND #PWR11
+L GND #PWR09
 U 1 1 50D12D5D
 P 5650 5650
-F 0 "#PWR11" H 5650 5650 30  0001 C CNN
+F 0 "#PWR09" H 5650 5650 30  0001 C CNN
 F 1 "GND" H 5650 5580 30  0001 C CNN
 	1    5650 5650
@@
 $EndComp
 $Comp
-L VCC #PWR10
+L VCC #PWR010
 U 1 1 50D12D63
 P 5650 2150
-F 0 "#PWR10" H 5650 2250 30  0001 C CNN
+F 0 "#PWR010" H 5650 2250 30  0001 C CNN
 F 1 "VCC" H 5650 2250 30  0000 C CNN
 	1    5650 2150
@@
 $EndComp
 $Comp
-L GND #PWR9
+L GND #PWR011
 U 1 1 50D12D8D
 P 2700 3500
-F 0 "#PWR9" H 2700 3500 30  0001 C CNN
+F 0 "#PWR011" H 2700 3500 30  0001 C CNN
 F 1 "GND" H 2700 3430 30  0001 C CNN
 	1    2700 3500
@@
 $EndComp
 $Comp
-L GND #PWR12
+L GND #PWR012
 U 1 1 50D12D93
 P 6300 3250
-F 0 "#PWR12" H 6300 3250 30  0001 C CNN
+F 0 "#PWR012" H 6300 3250 30  0001 C CNN
 F 1 "GND" H 6300 3180 30  0001 C CNN
 	1    6300 3250
@@
 $EndComp
 Wire Wire Line
-	5650 2150 5650 2500
-Wire Wire Line
-	5650 2500 5650 3200
+	5650 2150 5650 3200
 Wire Wire Line
 	5650 5300 5650 5650
@@
 	4200 2650 4200 2500
 Wire Wire Line
-	4200 2500 5650 2500
-Wire Wire Line
-	5650 2500 6050 2500
-Wire Wire Line
-	6050 2500 6550 2500
+	4200 2500 6550 2500
 Connection ~ 5650 2500
 Wire Wire Line
-	4200 3150 4200 3250
-Wire Wire Line
-	4200 3250 4200 3500
-Wire Wire Line
-	3750 3500 4200 3500
-Wire Wire Line
-	4200 3500 4300 3500
+	4200 3150 4200 3500
+Wire Wire Line
+	3750 3500 4300 3500
 Connection ~ 4200 3500
 Wire Wire Line
@@
 	6300 3250 6300 3150
 Wire Wire Line
-	6050 3150 6300 3150
-Wire Wire Line
-	6300 3150 6550 3150
+	6050 3150 6550 3150
 Wire Wire Line
 	6050 3150 6050 3050
@@
 	8400 2650 8800 2650
 $Comp
-L VCC #PWR13
+L VCC #PWR013
 U 1 1 50D1A22B
 P 8800 2150
-F 0 "#PWR13" H 8800 2250 30  0001 C CNN
+F 0 "#PWR013" H 8800 2250 30  0001 C CNN
 F 1 "VCC" H 8800 2250 30  0000 C CNN
 	1    8800 2150
@@
 $EndComp
 $Comp
-L GND #PWR14
+L GND #PWR014
 U 1 1 50D1A23A
 P 8800 3050
-F 0 "#PWR14" H 8800 3050 30  0001 C CNN
+F 0 "#PWR014" H 8800 3050 30  0001 C CNN
 F 1 "GND" H 8800 2980 30  0001 C CNN
 	1    8800 3050
